File: HVI.kicad_sch (KiCad schematic)
At the start: 34 parts, among them J1 Conn_01x02, J2 Conn_01x02, J3 Conn_01x02, U1 VIPER06-SSOP-10

Commit message: changed C2, DNP for C6, added Fuse Clips F1.1 and F1.2
Parts:
- added F1.1, F1.2: Fuse Clips, -, symbol Connector:Conn_01x01_Socket
- C2: value 1 µF -> 100nF
- C6: now not fitted; now left out of the parts list
- F1: value ≤ 500 mA -> ≤ 500 mA, solder Fuse Clips F1.1 and F1.2 and insert F1
- R6: now left out of the parts list
Connections:
- net at F1.2, R1.2, R2.2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: now also F1.2.1 (Pin_1)
- net at F1.1, J2.1 (Pin_1), J2.2 (Pin_2): now also F1.1.1 (Pin_1)
Other:
- note added: "A cartridge fuse from a multimeter can be used too"
- note added: "Fuse clips"
- note added: "Note on C11 If it is intend to drive a large load, then you can use C11 instead."
- note added: "Note on JP1 If the output J1 is used, bridge the left and middle or right and middle pads together with solder in order to choose between direct connection or resistor in series for the output."
- note added: "Note on R6 and C6 Those are just for development. Leave those footprints empty."
- note added: "Note: F1 is made from three parts. F1.1 and F1.2 are the fuse clips for soldering. F1 is the fuse itself (insert into fuse clips)"
- note added: "≤ 500 mA"
- note removed: "A cartridge fuse from a multimeter can be used too ;)"
Changed lines of the file:
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@@
 	)
 	(junction
+		(at 32.385 33.02)
+		(diameter 0)
+		(color 0 0 0 0)
+	)
+	(junction
 		(at 62.865 63.5)
 		(diameter 0)
@@
 	)
 	(junction
+		(at 24.765 33.02)
+		(diameter 0)
+		(color 0 0 0 0)
+	)
+	(junction
 		(at 34.925 33.02)
 		(diameter 0)
@@
 		)
 	)
+	(text "Note on C11\nIf it is intend to drive a large load, \nthen you can use C11 instead."
+		(exclude_from_sim no)
+		(at 153.67 77.47 0)
+		(effects
+			(font
+				(size 0.6 0.6)
+				(thickness 0.2)
+				(bold yes)
+			)
+			(justify left bottom)
+		)
+	)
 	(text "I'm unsure why 700 V and 800 V look so different from the others.\nMight need to re-test when I got time :‘)"
 		(exclude_from_sim no)
@@
 	(text "HV-"
 		(exclude_from_sim no)
-		(at 15.621 81.026 0)
+		(at 15.875 81.28 0)
 		(effects
 			(font
@@
 		)
 	)
+	(text "≤ 500 mA"
+		(exclude_from_sim no)
+		(at 28.575 35.56 0)
+		(effects
+			(font
+				(size 0.8 0.8)
+			)
+		)
+	)
 	(text "Isolated output"
 		(exclude_from_sim no)
-		(at 133.985 90.932 0)
+		(at 133.985 90.805 0)
 		(effects
 			(font
@@
 		)
 	)
+	(text "Note on R6 and C6\nThose are just for development.\nLeave those footprints empty."
+		(exclude_from_sim no)
+		(at 54.61 80.01 0)
+		(effects
+			(font
+				(size 0.6 0.6)
+				(thickness 0.2)
+				(bold yes)
+			)
+			(justify left bottom)
+		)
+	)
 	(text "RC-Lowpass \nagainst ripple \nconducting \nback to TS\n\nTau = 20 µs"
 		(exclude_from_sim no)
-		(at 31.115 57.785 0)
+		(at 31.115 59.055 0)
 		(effects
 			(font
@@
 		)
 	)
+	(text "Note: F1 is made from three parts.\nF1.1 and F1.2 are the fuse clips for soldering.\nF1 is the fuse itself (insert into fuse clips)"
+		(exclude_from_sim no)
+		(at 12.7 44.45 0)
+		(effects
+			(font
+				(size 0.6 0.6)
+				(thickness 0.16)
+				(bold yes)
+			)
+			(justify left bottom)
+		)
+	)
 	(text "12 V"
 		(exclude_from_sim no)
@@
 	(text "alternative \nfootprint"
 		(exclude_from_sim no)
-		(at 163.83 88.011 0)
+		(at 163.83 88.265 0)
 		(effects
 			(font
@@
 		)
 	)
-	(text "A cartridge fuse\nfrom a multimeter \ncan be used too ;)"
+	(text "Note on JP1\nIf the output J1 is used, bridge the left and middle or right and middle pads together \nwith solder in order to choose between direct connection or resistor in series for the output."
 		(exclude_from_sim no)
-		(at 22.098 40.513 0)
+		(at 155.575 96.52 0)
+		(effects
+			(font
+				(size 0.6 0.6)
+			)
+			(justify left)
+		)
+	)
+	(text "Fuse clips"
+		(exclude_from_sim no)
+		(at 28.575 29.21 0)
+		(effects
+			(font
+				(size 0.6 0.6)
+			)
+		)
+	)
+	(text "A cartridge fuse\nfrom a multimeter \ncan be used too"
+		(exclude_from_sim no)
+		(at 22.86 40.64 0)
 		(effects
 			(font
@@
 	(text "HV+"
 		(exclude_from_sim no)
-		(at 15.621 29.464 0)
+		(at 15.875 29.21 0)
 		(effects
 			(font
@@
 		(unit 1)
 		(exclude_from_sim no)
-		(in_bom yes)
+		(in_bom no)
 		(on_board yes)
 		(dnp yes)
@@
 			)
 		)
-		(property "Value" "1 µF"
+		(property "Value" "100nF"
 			(at 83.185 64.7762 0)
 			(effects
@@
 	)
 	(symbol
+		(lib_id "Connector:Conn_01x01_Socket")
+		(at 32.385 27.94 90)
+		(unit 1)
+		(exclude_from_sim no)
+		(in_bom yes)
+		(on_board no)
+		(dnp no)
+		(property "Reference" "F1.2"
+			(at 30.734 26.9239 90)
+			(effects
+				(font
+					(size 1 1)
+				)
+				(justify right)
+			)
+		)
+		(property "Value" "Fuse Clips"
+			(at 34.29 29.8449 90)
+			(effects
+				(font
+					(size 1.27 1.27)
+				)
+				(justify right)
+				(hide yes)
+			)
+		)
+		(property "Footprint" "-"
+			(at 32.385 27.94 0)
+			(effects
+				(font
+					(size 1.27 1.27)
+				)
+				(hide yes)
+			)
+		)
+		(property "Datasheet" "https://www.mouser.de/ProductDetail/Littelfuse/01220083Z?qs=95aqoVzNh5YRvw7yc4yLmA%3D%3D"
+			(at 32.385 27.94 0)
+			(effects
+				(font
+					(size 1.27 1.27)
+				)
+				(hide yes)
+			)
+		)
+		(property "Description" "Generic connector, single row, 01x01, script generated"
+			(at 32.385 27.94 0)
+			(effects
+				(font
+					(size 1.27 1.27)
+				)
+				(hide yes)
+			)
+		)
+		(pin "1"
+		)
+		(instances
+			(project "HVI"
+				(path "/96589b0c-b051-494a-952b-1d85eb492735"
+					(reference "F1.2")
+					(unit 1)
+				)
+			)
+		)
+	)
+	(symbol
 		(lib_id "Device:D_Small")
 		(at 80.01 80.01 270)
@@
 		(unit 1)
 		(exclude_from_sim no)
-		(in_bom yes)
+		(in_bom no)
 		(on_board yes)
-		(dnp no)
+		(dnp yes)
 		(property "Reference" "C6"
 			(at 59.69 67.3162 0)
@@
 			)
 		)
-		(property "Value" "≤ 500 mA"
+		(property "Value" "≤ 500 mA, solder Fuse Clips F1.1 and F1.2 and insert F1"
 			(at 28.575 35.0774 90)
 			(effects
@@
 					(size 0.8 0.8)
 				)
+				(hide yes)
 			)
 		)
@@
 					(unit 1)
 				)
+			)
+		)
+	)
+	(symbol
+		(lib_id "Connector:Conn_01x01_Socket")
+		(at 24.765 27.94 90)
+		(unit 1)
+		(exclude_from_sim no)
+		(in_bom yes)
+		(on_board no)
+		(dnp no)
+		(property "Reference" "F1.1"
+			(at 23.114 26.9239 90)
+			(effects
+				(font
+					(size 1 1)
+				)
+				(justify right)
+			)
+		)
+		(property "Value" "Fuse Clips"
+			(at 26.67 29.8449 90)
+			(effects
+				(font
+					(size 1.27 1.27)
+				)
+				(justify right)
+				(hide yes)
+			)
+		)
+		(property "Footprint" "-"
+			(at 24.765 27.94 0)
+			(effects
+				(font
+					(size 1.27 1.27)
+				)
+				(hide yes)
+			)
+		)
+		(property "Datasheet" "https://www.mouser.de/ProductDetail/Littelfuse/01220083Z?qs=95aqoVzNh5YRvw7yc4yLmA%3D%3D"
+			(at 24.765 27.94 0)
+			(effects
+				(font
+					(size 1.27 1.27)
+				)
+				(hide yes)
+			)
+		)
+		(property "Description" "Generic connector, single row, 01x01, script generated"
+			(at 24.765 27.94 0)
+			(effects
+				(font
+					(size 1.27 1.27)
+				)
+				(hide yes)
+			)
+		)
+		(pin "1"
+		)
+		(instances
+			(project ""
+				(path "/96589b0c-b051-494a-952b-1d85eb492735"
+					(reference "F1.1")
+					(unit 1)
+				)

Commit message: fixed BOM error, added additional component URLs
Parts:
- C2: Manufacturer Number (none) -> GRM188R72A103MA01J
- C7: Manufacturer Number (none) -> C0603C223J3RACAUTO
- D1: Manufacturer Number US3M-13 -> VS-E7FX0212-M3/I
- F1: Manufacturer Number (none) -> 0ADAC0250-BE
- F1.1, F1.2: Manufacturer Number (none) -> 01220083Z
- JP1: Manufacturer Number (none) -> -; now not fitted
- PS1: Manufacturer Number (none) -> PEME1-S12-S5-S
- R1, R2, R3: Manufacturer Number PEME1-S12-S5-S -> KTR18EZPF2700
- R4: Manufacturer Number (none) -> CRCW06031K00FKEE
- R5: Manufacturer Number (none) -> AC0603FR-0727KL
- R6: Manufacturer Number (none) -> -
- R7: Manufacturer Number (none) -> AC0603JR-0710KL
- R8: Manufacturer Number (none) -> AC0603FR-10150RL
Changed lines of the file:
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@@
 			)
 		)
-		(property "Manufacturer Number" ""
+		(property "Manufacturer Number" "-"
 			(at 59.055 63.5 0)
 			(effects
@@
 			)
 		)
-		(property "Datasheet" "-"
+		(property "Datasheet" "https://www.mouser.de/ProductDetail/YAGEO/AC0603JR-0710KL?qs=cGU37fGUGy9YzDGDQHkl5g%3D%3D"
 			(at 74.295 69.215 0)
 			(effects
@@
 			)
 		)
-		(property "Manufacturer Number" ""
+		(property "Manufacturer Number" "AC0603JR-0710KL"
 			(at 74.295 69.215 0)
 			(effects
@@
 			)
 		)
-		(property "Datasheet" "-"
+		(property "Datasheet" "https://www.mouser.de/ProductDetail/Murata-Electronics/GRM188R72A103MA01J?qs=QzBtWTOodeWXrWvHLobtrQ%3D%3D"
 			(at 80.01 63.5 0)
 			(effects
@@
 			)
 		)
-		(property "Manufacturer Number" ""
+		(property "Manufacturer Number" "GRM188R72A103MA01J"
 			(at 80.01 63.5 0)
 			(effects
@@
 			)
 		)
-		(property "Datasheet" "https://www.mouser.de/datasheet/2/670/peme1_s-1596077.pdf"
+		(property "Datasheet" "https://www.mouser.de/ProductDetail/CUI-Inc/PEME1-S12-S5-S?qs=iLbezkQI%252Bsil9QGLUwaYwA%3D%3D"
 			(at 141.605 81.915 0)
 			(effects
@@
 			)
 		)
-		(property "Manufacturer Number" ""
+		(property "Manufacturer Number" "PEME1-S12-S5-S "
 			(at 141.605 81.915 0)
 			(effects
@@
 			)
 		)
-		(property "Datasheet" "https://www.mouser.de/ProductDetail/CUI-Inc/PEME1-S12-S5-S?qs=iLbezkQI%252Bsil9QGLUwaYwA%3D%3D"
+		(property "Datasheet" "https://www.mouser.de/ProductDetail/ROHM-Semiconductor/KTR18EZPF2700?qs=493kPxzlxfI0Eh3cLVC%2FqA%3D%3D"
 			(at 38.735 45.72 0)
 			(effects
@@
 			)
 		)
-		(property "Manufacturer Number" "PEME1-S12-S5-S"
+		(property "Manufacturer Number" "KTR18EZPF2700"
 			(at 38.735 45.72 0)
 			(effects
@@
 		(in_bom yes)
 		(on_board yes)
-		(dnp no)
+		(dnp yes)
 		(property "Reference" "JP1"
 			(at 170.18 85.725 0)
@@
 			)
 		)
-		(property "Manufacturer Number" ""
+		(property "Manufacturer Number" "-"
 			(at 173.355 86.995 0)
 			(effects
@@
 			)
 		)
+		(property "Manufacturer Number" "01220083Z "
+			(at 32.385 27.94 0)
+			(effects
+				(font
+					(size 1.27 1.27)
+				)
+				(hide yes)
+			)
+		)
 		(pin "1"
 		)
@@
 			)
 		)
-		(property "Datasheet" "-"
+		(property "Datasheet" "https://www.mouser.de/ProductDetail/Vishay-Dale/CRCW06031K00FKEE?qs=%252B6g0mu59x7JNM5l%252Bg7fBgQ%3D%3D"
 			(at 68.58 59.055 0)
 			(effects
@@
 			)
 		)
-		(property "Manufacturer Number" ""
+		(property "Manufacturer Number" "CRCW06031K00FKEE"
 			(at 68.58 59.055 0)
 			(effects
@@
 			)
 		)
-		(property "Datasheet" "https://www.mouser.de/ProductDetail/CUI-Inc/PEME1-S12-S5-S?qs=iLbezkQI%252Bsil9QGLUwaYwA%3D%3D"
+		(property "Datasheet" "https://www.mouser.de/ProductDetail/ROHM-Semiconductor/KTR18EZPF2700?qs=493kPxzlxfI0Eh3cLVC%2FqA%3D%3D"
 			(at 38.735 33.02 0)
 			(effects
@@
 			)
 		)
-		(property "Manufacturer Number" "PEME1-S12-S5-S"
+		(property "Manufacturer Number" "KTR18EZPF2700"
 			(at 38.735 33.02 0)
 			(effects
@@
 			)
 		)
-		(property "Manufacturer Number" "US3M-13"
+		(property "Manufacturer Number" "VS-E7FX0212-M3/I "
 			(at 114.3 59.055 0)
 			(effects
@@
 			)
 		)
-		(property "Datasheet" "-"
+		(property "Datasheet" "https://www.mouser.de/ProductDetail/KEMET/C0603C223J3RACAUTO?qs=sSYV1F9c5cH7%2FAz%2FOpyTtQ%3D%3D"
 			(at 68.58 69.215 0)
 			(effects
@@
 			)
 		)
-		(property "Manufacturer Number" ""
+		(property "Manufacturer Number" "C0603C223J3RACAUTO "
 			(at 68.58 69.215 0)
 			(effects
@@
 			)
 		)
-		(property "Datasheet" "-"
+		(property "Datasheet" "https://www.mouser.de/ProductDetail/YAGEO/AC0603FR-0727KL?qs=yhV1fb9g%2FKYPMFaufpN2JA%3D%3D"
 			(at 74.295 59.055 0)
 			(effects
@@
 			)
 		)
-		(property "Manufacturer Number" ""
+		(property "Manufacturer Number" "AC0603FR-0727KL"
 			(at 74.295 59.055 0)
 			(effects
@@
 			)
 		)
-		(property "Datasheet" "https://www.mouser.de/ProductDetail/CUI-Inc/PEME1-S12-S5-S?qs=iLbezkQI%252Bsil9QGLUwaYwA%3D%3D"
+		(property "Datasheet" "https://www.mouser.de/ProductDetail/ROHM-Semiconductor/KTR18EZPF2700?qs=493kPxzlxfI0Eh3cLVC%2FqA%3D%3D"
 			(at 38.735 39.37 0)
 			(effects
@@
 			)
 		)
-		(property "Manufacturer Number" "PEME1-S12-S5-S"
+		(property "Manufacturer Number" "KTR18EZPF2700"
 			(at 38.735 39.37 0)
 			(effects
@@
 			)
 		)
-		(property "Datasheet" "-"
+		(property "Datasheet" "https://www.mouser.de/ProductDetail/YAGEO/AC0603FR-10150RL?qs=r5DSvlrkXmLR9P%2FIODCVmQ%3D%3D"
 			(at 173.355 79.375 0)
 			(effects
@@
 			)
 		)
-		(property "Manufacturer Number" ""
+		(property "Manufacturer Number" "AC0603FR-10150RL"
 			(at 173.355 79.375 0)
 			(effects
@@
 			)
 		)
-		(property "Datasheet" "https://www.reichelt.de/sicherung-6-3x32mm-1000v-0-25a-ar-ff-mms-p7600-p142812.html?&trstct=pol_4&nbc=1"
+		(property "Datasheet" "https://www.mouser.de/ProductDetail/Bel-Fuse/0ADAC0250-BE?qs=rrS6PyfT74etahbNPwSVLw%3D%3D"
 			(at 28.575 33.02 0)
 			(effects
@@
 			)
 		)
-		(property "Manufacturer Number" ""
+		(property "Manufacturer Number" "0ADAC0250-BE"
 			(at 28.575 33.02 0)
 			(effects
@@
 			(at 24.765 27.94 0)
 			(effects
+				(font
+					(size 1.27 1.27)
+				)
+				(hide yes)
+			)
+		)
+		(property "Manufacturer Number" "01220083Z "
+			(at 24.765 27.94 0)
+			(effects

Commit message: Added Mouser and LCSC Numbers. Updated to KiCad 9
Parts:
- C1: LCSC (none) -> C1919667; Mouser (none) -> 810-C5750X7R2J224K
- C10: LCSC (none) -> C22367827; Mouser (none) -> 81-GRM188R6YA106MA3J
- C2: LCSC (none) -> X; Mouser (none) -> 81-GRM188R72A103MA1J
- C3: LCSC (none) -> C913904; Mouser (none) -> 963-UMK107BBJ225KA-T
- C7: LCSC (none) -> C302020; Mouser (none) -> 80-C0603C223J3RAUTO
- C8, C9: LCSC (none) -> C2361249; Mouser (none) -> 963-E32MAB5476MPNDTJ
- D1: LCSC (none) -> X; Mouser (none) -> 78-VS-E7FX0212-M3/I
- D2, D6: LCSC (none) -> C2934846; Mouser (none) -> 621-US3M-13
- D3, D4, D5: LCSC (none) -> C5342734; Mouser (none) -> 604-APTD1608LSURCK
- D7: LCSC (none) -> C1972922; Mouser (none) -> 652-P6SMB13A
- F1: LCSC (none) -> X; Mouser (none) -> 530-0ADAC0250-BE
- F1.1, F1.2: LCSC (none) -> C206901; Mouser (none) -> 576-01220083Z
- J1, J2, J3: LCSC (none) -> C293740; Mouser (none) -> 538-43650-0215
- L1, L2: LCSC (none) -> X; Mouser (none) -> 652-SRR1208-472KL
- PS1: LCSC (none) -> X; Mouser (none) -> 490-PEME1-S12-S5-S
- R1, R2, R3: LCSC (none) -> C4466; Mouser (none) -> 755-KTR18EZPF2700
- R4: LCSC (none) -> C21190; Mouser (none) -> 71-CRCW06031K00FKEE
- R5: LCSC (none) -> C21190; Mouser (none) -> 603-AC0603FR-0727KL
- R7: LCSC (none) -> C25804; Mouser (none) -> 603-AC0603JR-0710KL
- R8: LCSC (none) -> C114608; Mouser (none) -> 603-AC0603FR-10150RL
- R9: LCSC (none) -> X; Mouser (none) -> 603-RC0201FR-074K7L
- U1: LCSC (none) -> C2845040; Mouser (none) -> 511-VIPER06XSTR
