File: HVI.kicad_pcb (KiCad board)
At the start: 2 copper layers, 48 x 48 mm, 47 parts, among them J1 Conn_01x02, J2 Conn_01x02, J3 Conn_01x02, U1 VIPer06-SSOP-10

Commit message: Changed D1, updated BOM
Parts:
- D1: value US3M-13 -> VS-E7FX0212-M3/I; footprint Diode_SMD:D_SMC -> Diode_SMD:D_SMF
- U1: value VIPer06-SSOP-10 -> VIPER06-SSOP-10
- moved D1 0.25 mm to (112.8, 92.9)
Routing:
- net Net-(D1-A): track 77.2 -> 79.4 mm
- net Net-(D1-K): track 6.27 -> 7.46 mm
Changed lines of the file:
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@@
 			)
 		)
-		(property "Value" "VIPer06-SSOP-10"
+		(property "Value" "VIPER06-SSOP-10"
 			(at 0 3.5 90)
 			(layer "F.Fab")
@@
 		)
 	)
-	(footprint "Diode_SMD:D_SMC"
+	(footprint "Diode_SMD:D_SMF"
 		(layer "F.Cu")
-		(at 112.57 92.92 180)
-		(descr "Diode SMC (DO-214AB)")
-		(tags "Diode SMC (DO-214AB)")
+		(at 112.824 92.92 180)
+		(descr "Diode SMF (DO-219AB), http://www.vishay.com/docs/95572/smf_do-219ab.pdf")
+		(tags "Diode SMF (DO-214AB)")
 		(property "Reference" "D1"
-			(at 0 0 0)
+			(at 0 -2 180)
 			(layer "F.SilkS")
 			(effects
@@
 			)
 		)
-		(property "Value" "US3M-13"
-			(at 0 4.2 0)
+		(property "Value" "VS-E7FX0212-M3/I"
+			(at 0 2 180)
 			(layer "F.Fab")
 			(effects
@@
 			)
 		)
-		(property "Footprint" "Diode_SMD:D_SMC"
+		(property "Footprint" "Diode_SMD:D_SMF"
 			(at 0 0 180)
 			(unlocked yes)
@@
 			)
 		)
-		(property "Datasheet" "https://www.diodes.com/assets/Datasheets/US3M.pdf"
+		(property "Datasheet" "https://www.mouser.de/ProductDetail/Vishay/VS-E7FX0212-M3-I?qs=sGAEpiMZZMtbRapU8LlZD8qu4xuMq4%252BSuyt6OIho4cA9a2wnVK4kLA%3D%3D"
 			(at 0 0 180)
 			(unlocked yes)
@@
 		(attr smd)
 		(fp_line
-			(start -4.91 3.25)
-			(end 3.6 3.25)
+			(start -2.36 1.01)
+			(end 1.4 1.01)
 			(stroke
 				(width 0.12)
@@
 		)
 		(fp_line
-			(start -4.91 3.25)
-			(end -4.91 -3.25)
+			(start -2.36 -1.01)
+			(end 1.4 -1.01)
 			(stroke
 				(width 0.12)
@@
 		)
 		(fp_line
-			(start -4.91 -3.25)
-			(end 3.6 -3.25)
+			(start -2.36 -1.01)
+			(end -2.36 1.01)
 			(stroke
 				(width 0.12)
@@
 		)
 		(fp_line
-			(start 4.9 3.35)
-			(end -4.9 3.35)
+			(start 2.35 1.15)
+			(end -2.35 1.15)
 			(stroke
 				(width 0.05)
@@
 		)
 		(fp_line
-			(start 4.9 -3.35)
-			(end 4.9 3.35)
+			(start 2.35 -1.15)
+			(end 2.35 1.15)
 			(stroke
 				(width 0.05)
@@
 		)
 		(fp_line
-			(start -4.9 3.35)
-			(end -4.9 -3.35)
+			(start -2.35 1.15)
+			(end -2.35 -1.15)
 			(stroke
 				(width 0.05)
@@
 		)
 		(fp_line
-			(start -4.9 -3.35)
-			(end 4.9 -3.35)
+			(start -2.35 -1.15)
+			(end 2.35 -1.15)
 			(stroke
 				(width 0.05)
@@
 		)
 		(fp_line
-			(start 3.55 3.1)
-			(end -3.55 3.1)
+			(start 1.4 0.9)
+			(end -1.4 0.9)
 			(stroke
 				(width 0.1)
@@
 		)
 		(fp_line
-			(start 3.55 -3.1)
-			(end 3.55 3.1)
+			(start 1.4 -0.9)
+			(end 1.4 0.9)
 			(stroke
 				(width 0.1)
@@
 		)
 		(fp_line
-			(start 3.55 -3.1)
-			(end -3.55 -3.1)
+			(start 1.4 -0.9)
+			(end -1.4 -0.9)
 			(stroke
 				(width 0.1)
@@
 		)
 		(fp_line
-			(start 0.50118 0.75032)
-			(end 0.50118 -0.79908)
+			(start 0.3 0.4)
+			(end 0.3 -0.4)
 			(stroke
 				(width 0.1)
@@
 		)
 		(fp_line
-			(start 0.50118 0.00102)
-			(end 1.4994 0.00102)
+			(start 0.3 0)
+			(end 0.9 0)
 			(stroke
 				(width 0.1)
@@
 		)
 		(fp_line
-			(start -0.64944 0.00102)
-			(end 0.50118 0.75032)
+			(start -0.3 0.00102)
+			(end 0.3 0.4)
 			(stroke
 				(width 0.1)
@@
 		)
 		(fp_line
-			(start -0.64944 0.00102)
-			(end 0.50118 -0.79908)
+			(start -0.3 0)
+			(end 0.3 -0.4)
 			(stroke
 				(width 0.1)
@@
 		)
 		(fp_line
-			(start -0.64944 0.00102)
-			(end -1.55114 0.00102)
+			(start -0.3 0)
+			(end -0.9 0)
 			(stroke
 				(width 0.1)
@@
 		)
 		(fp_line
-			(start -0.64944 -0.79908)
-			(end -0.64944 0.80112)
+			(start -0.3 -0.4)
+			(end -0.3 0.4)
 			(stroke
 				(width 0.1)
@@
 		)
 		(fp_line
-			(start -3.55 3.1)
-			(end -3.55 -3.1)
+			(start -1.4 0.9)
+			(end -1.4 -0.9)
 			(stroke
 				(width 0.1)
@@
 		)
 		(fp_text user "${REFERENCE}"
-			(at 0 -1.9 0)
+			(at 0 -2 180)
 			(layer "F.Fab")
 			(effects
@@
 		)
 		(pad "1" smd roundrect
-			(at -3.4 0 270)
-			(size 3.3 2.5)
+			(at -1.45 0 180)
+			(size 1.3 1.4)
 			(layers "F.Cu" "F.Paste" "F.Mask")
-			(roundrect_rratio 0.1)
+			(roundrect_rratio 0.1923076923)
 			(net 8 "Net-(D1-K)")
 			(pinfunction "K")
@@
 		)
 		(pad "2" smd roundrect
-			(at 3.4 0 270)
-			(size 3.3 2.5)
+			(at 1.45 0 180)
+			(size 1.3 1.4)
 			(layers "F.Cu" "F.Paste" "F.Mask")
-			(roundrect_rratio 0.1)
+			(roundrect_rratio 0.1923076923)
 			(net 9 "Net-(D1-A)")
 			(pinfunction "A")
 			(pintype "passive")
 		)
-		(model "${KICAD6_3DMODEL_DIR}/Diode_SMD.3dshapes/D_SMC.wrl"
+		(model "${KICAD8_3DMODEL_DIR}/Diode_SMD.3dshapes/D_SMF.wrl"
 			(offset
 				(xyz 0 0 0)
@@
 	)
 	(segment
-		(start 115.97 92.92)
+		(start 115.97 92.056)
+		(end 115.106 92.92)
+		(width 0.75)
+		(layer "F.Cu")
+		(net 8)
+	)
+	(segment
+		(start 115.97 89.916)
 		(end 115.97 88.4675)
 		(width 0.75)
@@
 	)
 	(segment
+		(start 115.97 89.916)
+		(end 115.97 92.056)
+		(width 0.75)
+		(layer "F.Cu")
+		(net 8)
+	)
+	(segment
+		(start 115.106 92.92)
+		(end 114.274 92.92)
+		(width 0.75)
+		(layer "F.Cu")
+		(net 8)
+	)
+	(segment
 		(start 81.42 79.175)
 		(end 75.5975 79.175)
@@
 		(start 105.865 92.92)
 		(end 103.82 90.875)
-		(width 2)
+		(width 1.5)
 		(layer "F.Cu")
 		(net 9)
@@
 	)
 	(segment
-		(start 109.17 92.92)
+		(start 111.374 92.92)
 		(end 105.865 92.92)
-		(width 2)
+		(width 1.5)
 		(layer "F.Cu")
 		(net 9)

Commit message: changed C2, DNP for C6, added Fuse Clips F1.1 and F1.2
Parts:
- C2: value 1 µF -> 100nF
- F1: value ≤ 500 mA -> ≤ 500 mA, solder Fuse Clips F1.1 and F1.2 and insert F1
Changed lines of the file:
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@@
 		(sheetname "Root")
 		(sheetfile "HVI.kicad_sch")
-		(attr smd dnp)
+		(attr smd exclude_from_bom dnp)
 		(fp_line
 			(start -0.254724 0.5225)
@@
 			)
 		)
-		(property "Value" "≤ 500 mA"
+		(property "Value" "≤ 500 mA, solder Fuse Clips F1.1 and F1.2 and insert F1"
 			(at 17.25 5.05 0)
 			(layer "F.Fab")
@@
 			)
 		)
-		(property "Value" "1 µF"
+		(property "Value" "100nF"
 			(at 0 1.43 90)
 			(layer "F.Fab")
@@
 			)
 		)
-		(property "Datasheet" "book"
+		(property "Datasheet" "-"
 			(at 0 0 90)
 			(unlocked yes)
@@
 			)
 		)
-		(property "Datasheet" "book"
+		(property "Datasheet" "-"
 			(at 0 0 -90)
 			(unlocked yes)
@@
 		(sheetname "Root")
 		(sheetfile "HVI.kicad_sch")
-		(attr smd)
+		(attr smd exclude_from_bom dnp)
 		(fp_line
 			(start -0.146267 0.51)
